File: elec/layout/default/show-and-tell.kicad_pcb (KiCad board)
At the start: 2 copper layers, 225.7 x 100.8 mm, 0 parts

Commit message: initial commit
Parts:
- added C1: 10V 10uF X5R ±10% 0603 Multilayer Ceramic Capacitors MLCC -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, lib:C0603, F.Cu at (137.0, 89.0)
- added C2: 10V 10uF X5R ±10% 0603 Multilayer Ceramic Capacitors MLCC -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, lib:C0603, F.Cu at (143.0, 87.6)
- added U1: , lib:SOT-25_L3.0-W1.6-P0.95-LS2.8-TL, F.Cu at (140.0, 89.5)
- added U2: , lib:WIFIM-SMD_61P-L16.6-W13.2-P0.80-ESP32-C6-MINI-1-N4, F.Cu at (152.0, 92.0)
- added U3: , lib:LGA-12_L2.0-W2.0-P0.50-BL, F.Cu at (164.6, 92.2)
Other:
- board size 225.7 x 100.8 mm -> 40 x 40 mm
- board text removed: "{{GITHASH}}"
